File: smc_board/smc_power_board/smc_power.kicad_sch (KiCad schematic)
At the start: 0 parts

Commit message: hw(power): WIP schematic updates (pre-restructure snapshot)
Parts:
- added C1, C10, C11, C12, C2, C3: 2.2uF, 100V, Capacitor_SMD:C_1206_3216Metric_Pad1.33x1.80mm_HandSolder, symbol Device:C
- added C13: 2.2nF, 25V, Capacitor_SMD:C_0805_2012Metric_Pad1.18x1.45mm_HandSolder, symbol Device:C
- added C14: 43pF, 25V, Capacitor_SMD:C_0805_2012Metric_Pad1.18x1.45mm_HandSolder, symbol Device:C
- added C15, C6: 100nF, 25V, Capacitor_SMD:C_0805_2012Metric_Pad1.18x1.45mm_HandSolder, symbol Device:C
- added C16: 47uF, 25V, Capacitor_THT:CP_Radial_D5.0mm_P2.50mm, symbol Device:C_Polarized
- added C17, C18: 1uF, Capacitor_SMD:C_0805_2012Metric_Pad1.18x1.45mm_HandSolder, symbol Device:C
- added C22, C23: 470uF 100V, Capacitor_THT:CP_Radial_D16.0mm_P7.50mm, symbol Device:C_Polarized
- added C24: 100nF 100V, Capacitor_SMD:C_0805_2012Metric_Pad1.18x1.45mm_HandSolder, symbol Device:C
- added C4: 5.1nF, 25V, Capacitor_SMD:C_0805_2012Metric_Pad1.18x1.45mm_HandSolder, symbol Device:C
- added C5: 24pF, 25V, Capacitor_SMD:C_0805_2012Metric_Pad1.18x1.45mm_HandSolder, symbol Device:C
- added C7: 68uF, 50V, Capacitor_THT:CP_Radial_D8.0mm_P3.50mm, symbol Device:C_Polarized
- added C8, C9: 10uF, 50V, Capacitor_SMD:C_1206_3216Metric_Pad1.33x1.80mm_HandSolder, symbol Device:C
- added D1: 100V 3A <= 850mV, Diode_SMD:D_SMB-SMC_Universal_Handsoldering, symbol Device:D_Schottky
- added D2: 100V 5A, Package_TO_SOT_SMD:TO-252-2, symbol Device:D_Schottky
- added D6: SMBJ58A, Diode_SMD:D_SMA-SMB_Universal_Handsoldering, symbol Device:D_Zener
- added D8: MBR10100, Step Motor Controller:TO508P482X997X1956-2P, symbol Step Motor Controller:MBR10100
- added F2: 100V 10A, Fuse:Fuseholder_Blade_Mini_Keystone_3568, symbol Device:Fuse
- added IC1: LM393DR2GH, Step Motor Controller:SOIC127P600X175-8N, symbol Step Motor Controller:LM393DR2GH
- added J1: Screw_Terminal_Input, TerminalBlock_Phoenix:TerminalBlock_Phoenix_MPT-0,5-2-2.54_1x02_P2.54mm_Horizontal, symbol Connector:Screw_Terminal_01x02
- added J2: Screw_Terminal_Output, symbol Connector:Screw_Terminal_01x05
- added L1: 68uH, Inductor_SMD:L_SXN_SMDRI125, symbol Device:L
- added L2: 22uH, Inductor_SMD:L_Chilisin_BMRF00101040, symbol Device:L
- added Q2: P40B10SL, Step Motor Controller:AOD4185, symbol Step Motor Controller:AOD4126
- added R1, R7: 523kR, Resistor_SMD:R_0805_2012Metric_Pad1.20x1.40mm_HandSolder, symbol Device:R
- added R10: 15.4kR, Resistor_SMD:R_0805_2012Metric_Pad1.20x1.40mm_HandSolder, symbol Device:R
- added R11: 60.4kR, Resistor_SMD:R_0805_2012Metric_Pad1.20x1.40mm_HandSolder, symbol Device:R
- added R12: 11.5kR, Resistor_SMD:R_0805_2012Metric_Pad1.20x1.40mm_HandSolder, symbol Device:R
- added R2, R8: 18.7kR, Resistor_SMD:R_0805_2012Metric_Pad1.20x1.40mm_HandSolder, symbol Device:R
- added R21: 97.6kR, Resistor_SMD:R_0805_2012Metric_Pad1.20x1.40mm_HandSolder, symbol Device:R
- added R22: 4.75kR, Resistor_SMD:R_0805_2012Metric_Pad1.20x1.40mm_HandSolder, symbol Device:R
- added R23: 1kR, Resistor_SMD:R_0805_2012Metric_Pad1.20x1.40mm_HandSolder, symbol Device:R
- added R24: 243kR, Resistor_SMD:R_0805_2012Metric_Pad1.20x1.40mm_HandSolder, symbol Device:R
- added R25: 10kR, Resistor_SMD:R_0805_2012Metric_Pad1.20x1.40mm_HandSolder, symbol Device:R
- added R26: 220R, Resistor_SMD:R_0805_2012Metric_Pad1.20x1.40mm_HandSolder, symbol Device:R
- added R27: 100k, Resistor_SMD:R_0805_2012Metric_Pad1.20x1.40mm_HandSolder, symbol Device:R
- added R28: 33R >=10W, Resistor_THT:R_Axial_DIN0516_L15.5mm_D5.0mm_P25.40mm_Horizontal, symbol Device:R
- added R3, R9: 267kR, Resistor_SMD:R_0805_2012Metric_Pad1.20x1.40mm_HandSolder, symbol Device:R
- added R4: 36.5kR, Resistor_SMD:R_0805_2012Metric_Pad1.20x1.40mm_HandSolder, symbol Device:R
- added R5: 348kR, Resistor_SMD:R_0805_2012Metric_Pad1.20x1.40mm_HandSolder, symbol Device:R
- added R6: 12kR, Resistor_SMD:R_0805_2012Metric_Pad1.20x1.40mm_HandSolder, symbol Device:R
- added U1, U2: TPS54360DDA, Package_SO:TI_SO-PowerPAD-8_ThermalVias, symbol Regulator_Switching:TPS54360DDA
- added U3: AP2112K-3.3, Package_TO_SOT_SMD:SOT-23-5, symbol Regulator_Linear:AP2112K-3.3
- added U6: TL431D, Package_SO:SOIC-8_3.9x4.9mm_P1.27mm, symbol Reference_Voltage:TL431D
Connections:
- new net: R23.1, U6.2 (A), U6.3 (A), U6.6 (A), U6.7 (A)
- new net: C15.2, D2.1 (K), L2.1, U2.8 (SW)
- new net: C5.1, R4.1, U1.6 (COMP)
- new net: C15.1, U2.1 (BOOT)
- new net: IC1.1 (OUTPUT_A), R24.2, R25.2, R26.1
- new net: Q2.1 (G), R26.2, R27.1
- new net: Q2.2 (D), R28.2
- new net: IC1.3 (INPUT_A_2), R21.2, R22.1, R24.1
- new net: R7.2, R8.1, U2.3 (EN)
- new net: C14.1, R10.1, U2.6 (COMP)
- new net: C4.1, R4.2
- new net: IC1.2 (INPUT_A_1), U6.8 (REF)
- new net: C13.1, R10.2
- new net: C6.1, U1.1 (BOOT)
- new net: R1.2, R2.1, U1.3 (EN)
- new net: R3.1, U1.4 (RT/CLK)
- new net: C6.2, D1.1 (K), L1.1, U1.8 (SW)
- new net: D8.2 (A), F2.2
- new net: R9.1, U2.4 (RT/CLK)
- new net +24V: C7.1, C8.1, C9.1, J2.4 (Pin_4), L1.2, R5.1
- new net +3V3: C18.1, J2.2 (Pin_2), U3.5 (VOUT)
- new net +48V: F2.1, J1.2 (Pin_2)
- new net +5V: C16.1, C17.1, C24.2, IC1.6 (INPUT_B_2), IC1.8 (VCC), J2.3 (Pin_3), L2.2, R11.1, R23.2, R25.1, U3.1 (VIN), U3.3 (EN)
- new net +VM: C1.1, C10.1, C11.1, C12.1, C2.1, C22.1, C23.1, C3.1, D6.1 (K), D8.1 (K), J2.5 (Pin_5), R1.1, R21.1, R28.1, R7.1, U1.2 (VIN), U2.2 (VIN)
- new net FB_24V: R5.2, R6.1, U1.5 (FB)
- new net FB_5V: R11.2, R12.1, U2.5 (FB)
- new net GND: C1.2, C10.2, C11.2, C12.2, C13.2, C14.2, C16.2, C17.2, C18.2, C2.2, C22.2, C23.2, C24.1, C3.2, C4.2, C5.2, C7.2, C8.2, C9.2, D1.2 (A), D2.2 (A), D6.2 (A), IC1.4 (GND), IC1.5 (INPUT_B_1), J1.1 (Pin_1), J2.1 (Pin_1), Q2.3 (S), R12.2, R2.2, R22.2, R27.2, R3.2, R6.2, R8.2, R9.2, U1.7 (GND), U1.9 (GNDPAD), U2.7 (GND), U2.9 (GNDPAD), U3.2 (GND), U6.1 (K)
- no-connect marks 0 -> 1
Other:
- note added: "24V Buck Converter"
- note added: "3V3 LDO"
- note added: "5V Buck Converter"
- note added: "Brake Chopper"
- note added: "C17, C18 -> 16V"
