File: hardware/power/smc_power.kicad_sch (KiCad schematic)
At the start: 102 parts, among them IC1 LM393DR2GH, J1 Screw_Terminal_01x02, J2 48V Input, J3 48V Output, J4 24V Brake Output, J5 Logic Output, Q1 P40B10SL, U1 TPS54360DDA, U2 AP2112K-3.3, U3 TPS54360DDA, U4 TPS16630PWPR, U5 MCP1416, U6 TL431B_C54830630, U7 L78L12_SOT89

Commit message: hw(power): board outline, mounting holes, zones, floorplan and chopper/buck/LDO layout, refs #39 #40 #41 #42 #43
Co-Authored-By: Claude Opus 5.5 <noreply@anthropic.com>
Claude-Session: https://claude.ai/code/session_01SoMHYQYx4yCFML8vht6Kpa
Parts:
- D2: value 100V 5A -> SS510; footprint Package_TO_SOT_SMD:TO-252-2 -> Diode_SMD:D_SMA; LCSC (none) -> C18199171
Changed lines of the file:
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@@
 			)
 		)
-		(property "Value" "100V 5A"
+		(property "Value" "SS510"
 			(at 162.56 177.4824 90)
 			(show_name no)
@@
 			)
 		)
-		(property "Footprint" "Package_TO_SOT_SMD:TO-252-2"
+		(property "Footprint" "Diode_SMD:D_SMA"
 			(at 160.02 176.53 0)
 			(hide yes)
@@
 			)
 		)
-		(property "Datasheet" ""
+		(property "Datasheet" "https://wmsc.lcsc.com/wmsc/upload/file/pdf/v2/lcsc/2310131745_hongjiacheng-SS510_C18199171.pdf"
 			(at 160.02 176.53 0)
 			(hide yes)
@@
 			)
 		)
-		(property "Description" "Schottky diode"
+		(property "Description" "100V 5A Schottky, SMA (DO-214AC) - 5V buck catch diode, same part as D5"
+			(at 160.02 176.53 0)
+			(hide yes)
+			(show_name no)
+			(do_not_autoplace no)
+			(effects
+				(font
+					(size 1.27 1.27)
+				)
+			)
+		)
+		(property "LCSC" "C18199171"
 			(at 160.02 176.53 0)
 			(hide yes)
@@
 			(show_name no)
 			(do_not_autoplace no)
+			(effects
+				(font
+					(size 1.27 1.27)
+				)
+			)
+		)
+		(property "Description" ""
+			(at 318.77 227.33 0)
+			(show_name no)
+			(do_not_autoplace no)

Commit message: hw(power): LCSC part numbers for 67 parts, 0.1% R13/R17, R14 1% (hysteresis), refs #48
Co-Authored-By: Claude Opus 5.5 <noreply@anthropic.com>
Claude-Session: https://claude.ai/code/session_01SoMHYQYx4yCFML8vht6Kpa
Parts:
- C1, C12, C23, C25: LCSC (none) -> C49678
- C10: LCSC (none) -> C113827
- C11: LCSC (none) -> C1750
- C13, C14, C15, C2, C3, C4: LCSC (none) -> C577211
- C16, C27: LCSC (none) -> C5341638
- C17: LCSC (none) -> C107112
- C18: LCSC (none) -> C376967
- C19: LCSC (none) -> C106243
- C20, C21: LCSC (none) -> C49256827
- C22: LCSC (none) -> C309049
- C24: LCSC (none) -> C354262
- C26, C5, C6: LCSC (none) -> C28323
- C7: LCSC (none) -> C724604
- C8, C9: LCSC (none) -> C5449000
- D1: LCSC (none) -> C14281
- D10, D11, D6, D7, D8, D9: LCSC (none) -> C2297
- D13: LCSC (none) -> C84256
- D3: LCSC (none) -> C26327
- D4: LCSC (none) -> C284023
- IC1: LCSC (none) -> C7955
- J5: LCSC (none) -> C157991
- L1: LCSC (none) -> C5183009
- L2: LCSC (none) -> C5174472
- R1, R7: LCSC (none) -> C228890
- R10: LCSC (none) -> C2933442
- R11, R5: LCSC (none) -> C17499
- R12: LCSC (none) -> C17418
- R13: LCSC (none) -> C5266156; Tolerance (none) -> 0.1%
- R14: LCSC (none) -> C2930186; Tolerance (none) -> 1%
- R15, R20: LCSC (none) -> C17414
- R17: LCSC (none) -> C2692699; Tolerance (none) -> 0.1%
- R18: LCSC (none) -> C17415
- R19: LCSC (none) -> C17513
- R2: LCSC (none) -> C400703
- R3, R9: LCSC (none) -> C104164
- R31: LCSC (none) -> C3013231
- R33: LCSC (none) -> C2933438
- R4: LCSC (none) -> C2999585
- R6: LCSC (none) -> C17444
- R8: LCSC (none) -> C2933477
- U1, U3: LCSC (none) -> C44377
- U2: LCSC (none) -> C51118
- U5: LCSC (none) -> C83775
- U7: LCSC (none) -> C69601
