File: hardware/power/smc_power.kicad_sch (KiCad schematic)
At the start: 102 parts, among them IC1 LM393DR2GH, J1 Screw_Terminal_01x02, J2 48V Input, J3 48V Output, J4 24V Brake Output, J5 Logic Output, Q1 P40B10SL, U1 TPS54360DDA, U2 AP2112K-3.3, U3 TPS54360DDA, U4 TPS16630PWPR, U5 MCP1416, U6 TL431B_C54830630, U7 L78L12_SOT89

Commit message: hw(power): R21 -> MF72 5D13 (fits 7.5 mm footprint), Q1 -> AOD4126, refs #48
Co-Authored-By: Claude Opus 5.5 <noreply@anthropic.com>
Claude-Session: https://claude.ai/code/session_01SoMHYQYx4yCFML8vht6Kpa
Parts:
- Q1: value P40B10SL -> AOD4126; LCSC (none) -> C457934
- R21: value NTC_5_20 -> MF72 5D13; LCSC C122780 -> C72683; Manufacturer Part MF72 5D11 -> MF72 5D13
Changed lines of the file:
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@@
 			)
 		)
-		(property "Value" "P40B10SL"
+		(property "Value" "AOD4126"
 			(at 233.68 251.4599 0)
 			(show_name no)
@@
 			)
 		)
+		(property "LCSC" "C457934"
+			(at 233.68 251.4599 0)
+			(hide yes)
+			(show_name no)
+			(do_not_autoplace no)
+			(effects
+				(font
+					(size 1.27 1.27)
+				)
+			)
+		)
 		(pin "3"
 		)
@@
 			)
 		)
-		(property "Value" "NTC_5_20"
+		(property "Value" "MF72 5D13"
 			(at 40.64 238.76 0)
 			(show_name no)
@@
 			)
 		)
-		(property "Datasheet" "https://www.lcsc.com/datasheet/lcsc_datasheet_1810170717_Nanjing-Shiheng-Elec-MF72-5D11_C72676.pdf"
+		(property "Datasheet" "https://www.lcsc.com/product-detail/C72683.html"
 			(at 40.64 242.57 0)
 			(hide yes)
@@
 			)
 		)
-		(property "Description" "-40℃~+170℃ 2800K 3W 4A 5Ω 7.5mm ±10% 插件,P=7.5mm NTC Thermistors ROHS"
+		(property "Description" "NTC inrush limiter 5 Ohm, 5 A, 4 W, disc D13 mm, P=7.5 mm (MF72 5D13)"
 			(at 40.64 242.57 0)
 			(hide yes)
@@
 			)
 		)
-		(property "LCSC" "C122780"
+		(property "LCSC" "C72683"
 			(at 40.64 242.57 0)
 			(hide yes)
@@
 			)
 		)
-		(property "Manufacturer Part" "MF72 5D11"
+		(property "Manufacturer Part" "MF72 5D13"
 			(at 40.64 242.57 0)
 			(hide yes)

Commit message: hw(power): readable part values (LED colour, connector/fuse part numbers); silkscreen labels kept as text, refs #48
Co-Authored-By: Claude Opus 5.5 <noreply@anthropic.com>
Claude-Session: https://claude.ai/code/session_01SoMHYQYx4yCFML8vht6Kpa
Parts:
- D1: value 100V 3A <= 850mV -> SS310B
- D10: value +5V -> LED green 0805
- D11: value +3V3 -> LED green 0805
- D13: value 24V BRK FLT -> LED red 0805
- D3: value MBR10100 -> MBR10100G
- D6: value +48V -> LED green 0805
- D7: value +VM -> LED green 0805
- D8: value +24V -> LED green 0805
- D9: value +12V -> LED green 0805
- F1: value 100V 10A -> Keystone 3568 + 10A mini fuse
- IC1: value LM393DR2GH -> LM393DR2G
- J1: value Screw_Terminal_01x02 -> KF128-5.08-2P
- J2: value 48V Input -> XT60PW-M
- J3: value 48V Output -> XT30PW-F
- J4: value 24V Brake Output -> B2P-VH
- J5: value Logic Output -> B5B-XH-A
- U6: value TL431B_C54830630 -> TL431B
- U7: value L78L12_SOT89 -> L78L12ACUTR
Changed lines of the file:
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@@
 			)
 		)
-		(property "Value" "+3V3"
+		(property "Value" "LED green 0805"
 			(at 386.08 124.7776 90)
 			(show_name no)
@@
 			)
 		)
-		(property "Value" "48V Input"
+		(property "Value" "XT60PW-M"
 			(at 21.844 26.924 90)
 			(show_name no)
@@
 			)
 		)
-		(property "Value" "LM393DR2GH"
+		(property "Value" "LM393DR2G"
 			(at 132.08 226.06 0)
 			(show_name no)
@@
 			)
 		)
-		(property "Value" "Logic Output"
+		(property "Value" "B5B-XH-A"
 			(at 87.63 30.48 90)
 			(show_name no)
@@
 			)
 		)
-		(property "Value" "Screw_Terminal_01x02"
+		(property "Value" "KF128-5.08-2P"
 			(at 245.11 236.2199 0)
 			(hide yes)
@@
 			)
 		)
-		(property "Value" "100V 10A"
+		(property "Value" "Keystone 3568 + 10A mini fuse"
 			(at 41.91 220.98 90)
 			(show_name no)
@@
 			)
 		)
-		(property "Value" "100V 3A <= 850mV"
+		(property "Value" "SS310B"
 			(at 163.83 113.9824 90)
 			(show_name no)
@@
 			)
 		)
-		(property "Value" "TL431B_C54830630"
+		(property "Value" "TL431B"
 			(at 98.044 265.176 0)
 			(show_name no)
@@
 			)
 		)
-		(property "Value" "24V Brake Output"
+		(property "Value" "B2P-VH"
 			(at 62.484 27.178 90)
 			(show_name no)
@@
 			)
 		)
-		(property "Value" "24V BRK FLT"
+		(property "Value" "LED red 0805"
 			(at 398.78 128.5874 90)
 			(show_name no)
@@
 			)
 		)
-		(property "Value" "+24V"
+		(property "Value" "LED green 0805"
 			(at 355.6 124.7776 90)
 			(show_name no)
@@
 			)
 		)
-		(property "Value" "L78L12_SOT89"
+		(property "Value" "L78L12ACUTR"
 			(at 275.59 163.83 0)
 			(show_name no)
@@
 			)
 		)
-		(property "Value" "48V Output"
+		(property "Value" "XT30PW-F"
 			(at 42.164 26.924 90)
 			(show_name no)
@@
 			)
 		)
-		(property "Value" "MBR10100"
+		(property "Value" "MBR10100G"
 			(at 25.4 234.9499 90)
 			(show_name no)
@@
 			)
 		)
-		(property "Value" "+48V"
+		(property "Value" "LED green 0805"
 			(at 334.01 124.7776 90)
 			(show_name no)
@@
 			)
 		)
-		(property "Value" "+5V"
+		(property "Value" "LED green 0805"
 			(at 375.92 124.7776 90)
 			(show_name no)
@@
 			)
 		)
-		(property "Value" "+VM"
+		(property "Value" "LED green 0805"
 			(at 345.44 124.7776 90)
 			(show_name no)
@@
 			)
 		)
-		(property "Value" "+12V"
+		(property "Value" "LED green 0805"
 			(at 365.76 124.7776 90)
 			(show_name no)
